File: flyback-conv.sch (KiCad schematic (older format))
At the start: 1 part

Commit message: added PDF of many components and completed main schematic
Parts:
- removed R1: 20k, Resistor_SMD:R_0603_1608Metric, symbol Device:R
- added C?: 82uF, Capacitor_THT:CP_Radial_D18.0mm_P7.50mm, symbol Device:CP
- added C?: 0.47uF, Capacitor_SMD:C_1812_4532Metric, symbol Device:C
- added C? (x2): 0.22uF/500V, Capacitor_SMD:C_1812_4532Metric, symbol Device:C
- added C? (x5): 0.022uF, Capacitor_SMD:C_0603_1608Metric, symbol Device:C
- added C? (x2): 3.3pF, Capacitor_SMD:C_0603_1608Metric, symbol Device:C
- added C? (x3): 0.01uF, Capacitor_SMD:C_0603_1608Metric, symbol Device:C
- added C?: 2200pF, Capacitor_SMD:C_0603_1608Metric, symbol Device:C
- added C?: 22pF, Capacitor_SMD:C_0603_1608Metric, symbol Device:C
- added C?: 12pF, Capacitor_SMD:C_0603_1608Metric, symbol Device:C
- added C? (x2): 0.1uF, Capacitor_SMD:C_0603_1608Metric, symbol Device:C
- added C?: 4.7uF, Capacitor_SMD:C_0805_2012Metric, symbol Device:C
- added C?: 1uF, Capacitor_SMD:C_0603_1608Metric, symbol Device:C
- added C? (x2): 220pF, Capacitor_SMD:C_0603_1608Metric, symbol Device:C
- added C? (x2): 0.47uF, Capacitor_SMD:C_0805_2012Metric, symbol Device:C
- added C?: 4700pF, Capacitor_SMD:C_0603_1608Metric, symbol Device:C
- added C?: 2200pF/250V, Capacitor_SMD:C_2220_5650Metric, symbol Device:C
- added D?: KBP06G, custom-footprint:VISHAY_2KBP, symbol Device:D_Bridge_+AA-
- added D?: RFU02VSM6S, custom-footprint:TUMD2SM, symbol Device:D
- added D? (x2): CZRU52C2, Diode_SMD:D_SOD-523, symbol Device:D_Zener
- added D? (x2): CZRU52C6V2, Diode_SMD:D_SOD-523, symbol Device:D_Zener
- added D?: SDM03U40-7, Diode_SMD:D_SOD-523, symbol Device:D_Schottky
- added D?: BZT52C22T-7, Diode_SMD:D_SOD-523, symbol Device:D_Zener
- added D?: CDSOD323-T24S, Diode_SMD:D_SOD-323, symbol Device:D_Zener
- added D? (x2): CSFMT108-HF, Diode_SMD:D_SOD-123, symbol Device:D
- added D?: BAV21W-7-F, Diode_SMD:D_SOD-123, symbol Device:D
- added D?: MMSZ5248B-7-F, Diode_SMD:D_SOD-123, symbol Device:D_Zener
- added F?: Fuse, Fuse:Fuse_Littlefuse_395Series, symbol Device:Fuse
- added FL?: 20mH, Inductor_THT:L_CommonMode_Wuerth_WE-CMB-S, symbol custom-lib:EMI_FILTER
- added J? (x2): HOLE, Connector_Pin:Pin_D1.0mm_L10.0mm, symbol Connector:Conn_01x01_Female
- added Q?: DMP510DL, Package_TO_SOT_SMD:SOT-23, symbol Device:Q_PMOS_GSD
- added Q? (x2): 2N7002KW, Package_TO_SOT_SMD:SOT-323_SC-70, symbol Device:Q_NMOS_GSD
- added Q?: BSS126H6906, Package_TO_SOT_SMD:SOT-23, symbol Device:Q_NMOS_GSD
- added Q?: PGA26E07, custom-footprint:PANASONIC_PGA26E07BA, symbol custom-lib:PGA26E07
- added Q?: MMBTA42, Package_TO_SOT_SMD:SOT-23, symbol Device:Q_NPN_BEC
- added R? (x2): 1M, Resistor_SMD:R_0805_2012Metric, symbol Device:R
- added R? (x6): 10R, Resistor_SMD:R_0603_1608Metric, symbol Device:R
- added R? (x2): 10k, Resistor_SMD:R_0603_1608Metric, symbol Device:R
- added R?: 2R, Resistor_SMD:R_0603_1608Metric, symbol Device:R
- added R?: 100k, Resistor_SMD:R_0603_1608Metric, symbol Device:R
- added R?: 1.6k, Resistor_SMD:R_0603_1608Metric, symbol Device:R
- added R?: 0.18R, Resistor_SMD:R_1206_3216Metric, symbol Device:R
- added R?: 47.5k, Resistor_SMD:R_0603_1608Metric, symbol Device:R
- added R?: 121R, Resistor_SMD:R_0603_1608Metric, symbol Device:R
- added R? (x2): 1M, Resistor_SMD:R_0603_1608Metric, symbol Device:R
- added R?: 69.8k, Resistor_SMD:R_0603_1608Metric, symbol Device:R
- added R? (x2): 1R, Resistor_SMD:R_0805_2012Metric, symbol Device:R
- added R?: 191k, Resistor_SMD:R_0603_1608Metric, symbol Device:R
- added R?: 82.5k, Resistor_SMD:R_0603_1608Metric, symbol Device:R
- added R?: 221k, Resistor_SMD:R_0603_1608Metric, symbol Device:R
- added R?: 56.2k, Resistor_SMD:R_0603_1608Metric, symbol Device:R
- added R?: 22.1k, Resistor_SMD:R_0603_1608Metric, symbol Device:R
- added R?: 27k, Resistor_SMD:R_0603_1608Metric, symbol Device:R
- added R?: 562R, Resistor_SMD:R_0603_1608Metric, symbol Device:R
- added R?: 34k, Resistor_SMD:R_0603_1608Metric, symbol Device:R
- added R?: 11k, Resistor_SMD:R_0603_1608Metric, symbol Device:R
- added R?: 60.4k, Resistor_SMD:R_0603_1608Metric, symbol Device:R
- added R? (x2): 150k, Resistor_SMD:R_0603_1608Metric, symbol Device:R
- added T?: RM8, symbol custom-lib:RM8
- added TH?: 47k, Resistor_SMD:R_0603_1608Metric, symbol Device:Thermistor_NTC
- added U?: ISO7710, Package_SO:SOIC-8_3.9x4.9mm_P1.27mm, symbol custom-lib:ISO7710
- added U?: NV6115, symbol custom-lib:NV6115
- added U?: NV6117, symbol custom-lib:NV6115
- added U?: ATL431, Package_TO_SOT_SMD:SOT-23, symbol custom-lib:ATL431
- added U?: UCC28780, Package_DFN_QFN:QFN-16-1EP_3x3mm_P0.5mm_EP2.7x2.7mm_ThermalVias, symbol custom-lib:UCC28780
- added U?: AN34092B, Package_DFN_QFN:QFN-16-1EP_4x4mm_P0.65mm_EP2.7x2.7mm, symbol custom-lib:AN34092B
- added U?: SFH617A-1, Package_DIP:DIP-4_W7.62mm, symbol Isolator:SFH617A-1
Connections:
- net labels added: CS, CTL, DAUX2_2, Earth, F, FB, GND, INH, L, N, PWMH, PWML, RUN, S, VCC1, VCC2, VCCH, VCCL, VDD, VS, VSW, Vo, Vref
- wire segments 0 -> 326
- no-connect marks 0 -> 21

Commit message: fixed few lib componentes and screated PCB
Parts:
- added C1, C2: 2.2uF, Capacitor_SMD:C_0805_2012Metric, symbol Device:C
- added C10, C8, C9: 270uF, Capacitor_THT:CP_Radial_D8.0mm_P3.50mm, symbol Device:CP
- added C11: 0.01uF, Capacitor_SMD:C_0603_1608Metric, symbol Device:C
- added C12: 0.33uF, Capacitor_SMD:C_0603_1608Metric, symbol Device:C
- added C16: 6.8uF, Capacitor_SMD:C_0805_2012Metric, symbol Device:C
- added C26, C30, C32: 0.1uF, Capacitor_SMD:C_0603_1608Metric, symbol Device:C
- added C3: 220pF/250V, Capacitor_SMD:C_0603_1608Metric, symbol Device:C
- added C34: 0.22uF, Capacitor_SMD:C_0603_1608Metric, symbol Device:C
- added C4, C5: 33uF, Capacitor_SMD:C_1206_3216Metric, symbol Device:C
- added C42: 560pF, Capacitor_SMD:C_0603_1608Metric, symbol Device:C
- added C6, C7: 10uF, Capacitor_SMD:C_1206_3216Metric, symbol Device:C
- added D3: B340A-13-F, Diode_SMD:D_SMA, symbol Device:D_Schottky
- added D6: TPD1E05U06QDPYRQ, custom-lib:X1SON2, symbol Device:D_TVS_ALT
- added J3: USB_C_Receptacle, Connector_USB:USB_C_Receptacle_Amphenol_12401548E4-2A, symbol Connector:USB_C_Receptacle
- added L1: 0.68uH, Inductor_SMD:L_1206_3216Metric, symbol Device:L_Core_Iron
- added L2: 1uH, custom-lib:WURTH_7447462010, symbol Device:L_Core_Iron
- added Q1: BSC093N15NS5ATMA, Package_SON:VSONP-8-1EP_5x6_P1.27mm, symbol Device:Q_NMOS_SGD
- added Q2: CSD17578Q3, custom-lib:VSONP-8-1EP_3.3x3.3_P0.65mm, symbol Device:Q_NMOS_SGD
- added R1, R37: 100R, Resistor_SMD:R_0603_1608Metric, symbol Device:R
- added R10: 24.9R, Resistor_SMD:R_0603_1608Metric, symbol Device:R
- added R12: 0.005R, Resistor_SMD:R_1206_3216Metric, symbol Device:R
- added R2: 22R, Resistor_SMD:R_1206_3216Metric, symbol Device:R
- added R21, R39: 0R, Resistor_SMD:R_0603_1608Metric, symbol Device:R
- added R22: 2k, Resistor_SMD:R_0603_1608Metric, symbol Device:R
- added R25: 61.9k, Resistor_SMD:R_0603_1608Metric, symbol Device:R
- added R26: 90.9k, Resistor_SMD:R_0603_1608Metric, symbol Device:R
- added R3: 10R, Resistor_SMD:R_0603_1608Metric, symbol Device:R
- added R35: 100k, Resistor_SMD:R_0603_1608Metric, symbol Device:R
- added R36: 75k, Resistor_SMD:R_0603_1608Metric, symbol Device:R
- added R4: 1k, Resistor_SMD:R_0603_1608Metric, symbol Device:R
- added U1: UCC24612, Package_TO_SOT_SMD:SOT-23-5, symbol custom-lib:UCC24612
- added U6: TPS25740B, Package_DFN_QFN:QFN-24-1EP_4x4mm_P0.5mm_EP2.6x2.6mm, symbol custom-lib:TPS25740B
- D4: renamed from D?; footprint custom-footprint:TUMD2SM -> custom-lib:TUMD2SM
- D9: renamed from D?; footprint custom-footprint:VISHAY_2KBP -> custom-lib:VISHAY_2KBP
- Q8: renamed from Q?; footprint custom-footprint:PANASONIC_PGA26E07BA -> custom-lib:PANASONIC_PGA26E07BA
- U9: renamed from U?; footprint Package_DFN_QFN:QFN-16-1EP_4x4mm_P0.65mm_EP2.7x2.7mm -> Package_DFN_QFN:QFN-16-1EP_4x4mm_P0.65mm_EP2.5x2.5mm
- gave numbers to parts that had none: 88
Connections:
- net labels added: CC2, DVDD, GDNG, GDNS, ISNS, VBUS, Vaux
- wire segments 326 -> 484
- no-connect marks 21 -> 37
Other:
- note added: "CONTROL BOARD"
- note added: "MAIN BOARD"
- moved on the sheet: U7

Commit message: generated BOM v1.0, added some screenshots and added an alternative for the transformer
Parts:
- T1: value RM8 -> 150-2670; footprint (none) -> Transformer_THT:Transformer_37x44; Description RM8 Transformer -> Wurth ER28/14 Transformer, TO BE TESTED; MPN 750343793 -> 150-2670
- U1: Description Switching Controllers High-Frequency Multi-Mode Synchronous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 -> High-Frequency Multi-Mode Synchronous Rectifier Controller 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
- renumbered C13 to C11, C11 to C12, C14 to C13, C15 to C14, C17 to C15, C12 to C16, C18 to C17, C19 to C18, C20 to C19, C16 to C20, C27 to C26, C28 to C27, C29 to C28, C31 to C29, C33 to C30, C35 to C31, C36 to C32, C37 to C33, C26 to C34, C38 to C35, C30 to C36, C32 to C37, C34 to C38, C43 to C42, C44 to C43, C45 to C44, C42 to C45, D4 to D3, D5 to D4, D3 to D5, D7 to D6, D8 to D7, D9 to D8, D6 to D9, Q3 to Q2, Q4 to Q3, Q5 to Q4, Q2 to Q5, R3 to R10, R4 to R11, R14 to R12, R15 to R13, R10 to R14, R16 to R15, R17 to R16, R12 to R17, R23 to R21, R24 to R22, R27 to R23, R28 to R24, R29 to R25, R30 to R26, R21 to R27, R22 to R28, R31 to R29, R5 to R3, R32 to R30, R33 to R31, R34 to R32, R25 to R33, R26 to R34, R38 to R35, R40 to R36, R41 to R37, R42 to R38, R43 to R39, R6 to R4, R35 to R40, R36 to R41, R37 to R42, R44 to R43, R39 to R44, R7 to R5, R8 to R6, R9 to R7, R11 to R8, R13 to R9, U7 to U6, U6 to U7
